File: Hardware/Qwiic UV Sensor - ZOPT220x.brd (EAGLE design)
At the start: 25.4 x 25.4 mm, 17 parts, among them J2 SMD, J3 PTH, J4 SMD, U1 ZOPT220X

Commit message: Cleaning up file structure
Parts:
- J5: device SparkFun-Connectors:1X01NS_KIT -> SparkFun-Connectors:1X01_NO_SILK
Other:
- board text added: "ZOPT2201 UV Index Sensor"
- board text removed: "ZOPT220x UV Index Sensor"
Changed lines of the file:
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@@
 <grid distance="0.05" unitdist="inch" unit="inch" style="lines" multiple="1" display="yes" altdistance="0.005" altunitdist="inch" altunit="inch"/>
 <layers>
-<layer number="1" name="Top" color="4" fill="1" visible="yes" active="yes"/>
+<layer number="1" name="Top" color="4" fill="1" visible="no" active="yes"/>
 <layer number="2" name="Route2" color="1" fill="3" visible="no" active="no"/>
 <layer number="3" name="Route3" color="4" fill="3" visible="no" active="no"/>
@@
 <layer number="14" name="Route14" color="1" fill="6" visible="no" active="no"/>
 <layer number="15" name="Route15" color="4" fill="6" visible="no" active="no"/>
-<layer number="16" name="Bottom" color="1" fill="1" visible="yes" active="yes"/>
+<layer number="16" name="Bottom" color="1" fill="1" visible="no" active="yes"/>
 <layer number="17" name="Pads" color="2" fill="1" visible="yes" active="yes"/>
-<layer number="18" name="Vias" color="2" fill="1" visible="yes" active="yes"/>
-<layer number="19" name="Unrouted" color="6" fill="1" visible="yes" active="yes"/>
+<layer number="18" name="Vias" color="2" fill="1" visible="no" active="yes"/>
+<layer number="19" name="Unrouted" color="6" fill="1" visible="no" active="yes"/>
 <layer number="20" name="Dimension" color="15" fill="1" visible="yes" active="yes"/>
 <layer number="21" name="tPlace" color="16" fill="1" visible="yes" active="yes"/>
-<layer number="22" name="bPlace" color="14" fill="1" visible="yes" active="yes"/>
+<layer number="22" name="bPlace" color="14" fill="1" visible="no" active="yes"/>
 <layer number="23" name="tOrigins" color="15" fill="1" visible="yes" active="yes"/>
-<layer number="24" name="bOrigins" color="15" fill="1" visible="yes" active="yes"/>
+<layer number="24" name="bOrigins" color="15" fill="1" visible="no" active="yes"/>
 <layer number="25" name="tNames" color="7" fill="1" visible="no" active="yes"/>
 <layer number="26" name="bNames" color="7" fill="1" visible="no" active="yes"/>
-<layer number="27" name="tValues" color="7" fill="1" visible="no" active="yes"/>
+<layer number="27" name="tValues" color="7" fill="1" visible="yes" active="yes"/>
 <layer number="28" name="bValues" color="7" fill="1" visible="no" active="yes"/>
 <layer number="29" name="tStop" color="7" fill="3" visible="no" active="yes"/>
 <layer number="30" name="bStop" color="7" fill="6" visible="no" active="yes"/>
-<layer number="31" name="tCream" color="7" fill="4" visible="no" active="yes"/>
+<layer number="31" name="tCream" color="7" fill="4" visible="yes" active="yes"/>
 <layer number="32" name="bCream" color="7" fill="5" visible="no" active="yes"/>
 <layer number="33" name="tFinish" color="6" fill="3" visible="no" active="yes"/>
@@
 <text x="17.78" y="2.54" size="1.016" layer="22" font="vector" ratio="15" rot="MR90" align="center-left">!INT</text>
 <text x="7.62" y="2.54" size="1.016" layer="22" font="vector" ratio="15" rot="MR90" align="center-left">GND</text>
-<text x="12.827" y="22.86" size="1.016" layer="21" font="vector" ratio="15" rot="SR0" align="center">ZOPT220x
+<text x="12.827" y="22.86" size="1.016" layer="21" font="vector" ratio="15" rot="SR0" align="center">ZOPT2201
 UV Index Sensor</text>
-<text x="12.573" y="22.86" size="1.016" layer="22" font="vector" ratio="15" rot="SMR0" align="center">ZOPT220x
+<text x="12.573" y="22.86" size="1.016" layer="22" font="vector" ratio="15" rot="SMR0" align="center">ZOPT2201
 UV Index Sensor</text>
 <text x="2.413" y="1.27" size="1.27" layer="16" font="vector" ratio="15" rot="MR0" align="center">X01</text>
@@
 <element name="FRAME1" library="SparkFun-Aesthetics" package="CREATIVE_COMMONS" value="FRAME-LETTER" x="-20.32" y="-17.78"/>
 <element name="U$2" library="SparkX" package="SPARKX-MEDIUM" value="SPARKX-LOGO4" x="12.7" y="19.685"/>
-<element name="C4" library="SparkFun-Capacitors" package="0603" value="0.1uF" x="16.51" y="12.7" rot="R270">
+<element name="C4" library="SparkFun-Capacitors" package="0603" value="0.1uF" x="16.51" y="12.7" smashed="yes" rot="R270">
 <attribute name="PROD_ID" value="CAP-00810" x="16.51" y="12.7" size="1.778" layer="27" font="vector" ratio="15" rot="R270" display="off"/>
+<attribute name="NAME" x="17.272" y="12.7" size="0.6096" layer="25" font="vector" ratio="20" rot="R270" align="bottom-center"/>
+<attribute name="VALUE" x="15.748" y="12.7" size="0.6096" layer="27" font="vector" ratio="20" rot="R270" align="top-center"/>
 </element>
 <element name="J4" library="SparkX" package="1X04_1MM_RA" value="SMD" x="20.32" y="12.7" rot="R90"/>
 <element name="LOGO1" library="SparkFun-Aesthetics" package="OSHW-LOGO-MINI" value="OSHW-LOGOMINI" x="2.54" y="3.81" rot="MR0"/>
 <element name="U$1" library="SparkX" package="SPARKX-MEDIUM" value="SPARKX-LOGO4" x="12.7" y="19.685" rot="MR0"/>
-<element name="U1" library="SparkX" package="LGA6" value="ZOPT220X" x="12.7" y="12.7"/>
-<element name="J5" library="SparkFun-Connectors" package="1X01NS_KIT" value="" x="17.78" y="1.27"/>
+<element name="U1" library="SparkX" package="LGA6" value="ZOPT220X" x="12.7" y="12.7" smashed="yes">
+<attribute name="NAME" x="13.97" y="12.954" size="0.508" layer="25" ratio="15"/>
+<attribute name="VALUE" x="10.922" y="10.541" size="0.508" layer="27" ratio="15"/>
+</element>
+<element name="J5" library="SparkFun-Connectors" package="1X01_NO_SILK" value="" x="17.78" y="1.27"/>
 </elements>
 <signals>
